Commit message: new coke model added

File: urdf/coke_can.urdf (robot description, URDF)
Before this commit: robot coke_can_model, 1 links, 0 joints
Links:
- link coke_can: geometry collision mesh filename=package://pybullet_utils/meshes/coke_can.STL; visual mesh filename=package://pybullet_utils/meshes/coke_can.STL
